File: hand_pcb_rev2 - Copy/hand_pcb.sch (EAGLE design)
At the start: 66 parts

Commit message: added testpads for error pins on motor drivers
Parts:
- added IMF, PYF, TF: TESTPAD, 445-eagle-lib:TESTPAD
Connections:
- new net N$4: IMF.P$1, INDMID.NFAULT
- new net N$5: PKYRNG.NFAULT, PYF.P$1
- new net N$6: TF.P$1, THMB.NFAULT
Changed lines of the file:
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@@
 <part name="U$11" library="445-eagle-lib" deviceset="THRUHOLEI2C" device=""/>
 <part name="U$12" library="445-eagle-lib" deviceset="THRUHOLEI2C" device=""/>
+<part name="IMF" library="445-eagle-lib" deviceset="TESTPAD" device=""/>
+<part name="PYF" library="445-eagle-lib" deviceset="TESTPAD" device=""/>
+<part name="TF" library="445-eagle-lib" deviceset="TESTPAD" device=""/>
 </parts>
 <sheets>
@@
 <instance part="U$11" gate="G$1" x="203.2" y="149.86"/>
 <instance part="U$12" gate="G$1" x="236.22" y="149.86"/>
+<instance part="IMF" gate="G$1" x="185.42" y="106.68" rot="R180"/>
+<instance part="PYF" gate="G$1" x="185.42" y="55.88" rot="R180"/>
+<instance part="TF" gate="G$1" x="185.42" y="5.08" rot="R180"/>
 </instances>
 <busses>
@@
 </segment>
 </net>
+<net name="N$4" class="0">
+<segment>
+<pinref part="INDMID" gate="G$1" pin="NFAULT"/>
+<pinref part="IMF" gate="G$1" pin="P$1"/>
+<wire x1="180.34" y1="106.68" x2="185.42" y2="106.68" width="0.1524" layer="91"/>
+</segment>
+</net>
+<net name="N$5" class="0">
+<segment>
+<pinref part="PKYRNG" gate="G$1" pin="NFAULT"/>
+<pinref part="PYF" gate="G$1" pin="P$1"/>
+<wire x1="180.34" y1="55.88" x2="185.42" y2="55.88" width="0.1524" layer="91"/>
+</segment>
+</net>
+<net name="N$6" class="0">
+<segment>
+<pinref part="TF" gate="G$1" pin="P$1"/>
+<pinref part="THMB" gate="G$1" pin="NFAULT"/>
+<wire x1="185.42" y1="5.08" x2="180.34" y2="5.08" width="0.1524" layer="91"/>
+</segment>
+</net>

Commit message: added .1uF cap for io expander for stability - not fully needed but good practice
Parts:
- added C19: 0.1, rcl:C-USC0402
Connections:
- net +3V3: now also C19.1
- net GND: now also C19.2
Changed lines of the file:
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@@
 <part name="PYF" library="445-eagle-lib" deviceset="TESTPAD" device=""/>
 <part name="TF" library="445-eagle-lib" deviceset="TESTPAD" device=""/>
+<part name="C19" library="rcl" deviceset="C-US" device="C0402" value="0.1"/>
 </parts>
 <sheets>
@@
 <instance part="PYF" gate="G$1" x="185.42" y="55.88" rot="R180"/>
 <instance part="TF" gate="G$1" x="185.42" y="5.08" rot="R180"/>
+<instance part="C19" gate="G$1" x="66.04" y="-12.7"/>
 </instances>
 <busses>
@@
 <pinref part="SUPPLY7" gate="GND" pin="GND"/>
 <wire x1="78.74" y1="-17.78" x2="81.28" y2="-17.78" width="0.1524" layer="91"/>
+<pinref part="C19" gate="G$1" pin="2"/>
+<wire x1="66.04" y1="-17.78" x2="78.74" y2="-17.78" width="0.1524" layer="91"/>
+<junction x="78.74" y="-17.78"/>
 </segment>
 <segment>
@@
 <pinref part="+3V3" gate="G$1" pin="+3V3"/>
 <wire x1="78.74" y1="-15.24" x2="81.28" y2="-15.24" width="0.1524" layer="91"/>
-</segment>
-<segment>
+<pinref part="C19" gate="G$1" pin="1"/>
+<wire x1="73.66" y1="-10.16" x2="66.04" y2="-10.16" width="0.1524" layer="91"/>
+<wire x1="78.74" y1="-15.24" x2="73.66" y2="-15.24" width="0.1524" layer="91"/>
+<wire x1="73.66" y1="-15.24" x2="73.66" y2="-10.16" width="0.1524" layer="91"/>
+<junction x="78.74" y="-15.24"/>
+</segment>
+<segment>
